File: IOTV/pcb/IOTV_id5/IOTV.kicad_pcb (KiCad board)
At the start: 2 copper layers, 83.1 x 77.8 mm, 23 parts, among them J1 Screw_Terminal_01x02, J2 Screw_Terminal_01x02, J3 Conn_01x04, J4 Conn_01x04, J5 Conn_01x04, J6 Conn_01x05, K1 TIANBO-HJR-4102-L, Q1 MMBT3904, U1 ESP32_DevKit_V1_DOIT

Commit message: id-5 pcb
Routing:
- net Net-(D2-A): track 15.5 -> 21.7 mm
- net Net-(D1-A): track 16.4 -> 21.6 mm
- net SDA: track 125.9 -> 125.0 mm
- added copper zone on B.Cu, net ~220
