File: IOTV/pcb/IOTV_id5/IOTV.kicad_pcb (KiCad board)
At the start: 2 copper layers, 83.1 x 77.8 mm, 23 parts, among them J1 Screw_Terminal_01x02, J2 Screw_Terminal_01x02, J3 Conn_01x04, J4 Conn_01x04, J5 Conn_01x04, J6 Conn_01x05, K1 TIANBO-HJR-4102-L, Q1 MMBT3904, U1 ESP32_DevKit_V1_DOIT

Commit message: PCB id5
Parts:
- removed D1, D2, D3: LED, LED_SMD:LED_0603_1608Metric
- removed D5: SS26, Diode_SMD:D_SMB
- removed K1: TIANBO-HJR-4102-L, Relay_THT:Relay_SPDT_HJR-4102
- removed Q1: MMBT3904, Package_TO_SOT_SMD:SOT-23
- removed R3: 0R_0603, PCM_Resistor_SMD_AKL:R_1206_3216Metric
- added C1: C_Generic, Capacitor_SMD:C_1206_3216Metric, B.Cu at (121.7, 99.7)
- added C2: C_Generic, Capacitor_SMD:C_1206_3216Metric, B.Cu at (117.7, 99.7)
- added C3: C_Generic, Capacitor_SMD:C_1206_3216Metric, B.Cu at (123.7, 105.5)
- added C4: C_Generic, Capacitor_SMD:C_1206_3216Metric, B.Cu at (113.7, 99.8)
- added J7: JTAG, Connector_PinHeader_2.54mm:PinHeader_1x04_P2.54mm_Vertical, F.Cu at (157.2, 111.2)
- added J8: UART, Connector_PinHeader_2.54mm:PinHeader_1x04_P2.54mm_Vertical, F.Cu at (149.2, 111.2)
- added SW1: RST, Button_Switch_SMD:SW_SPST_TL3342, F.Cu at (147.2, 119.2)
- added SW2: Boot, Button_Switch_SMD:SW_SPST_TL3342, F.Cu at (157.2, 119.2)
- added U2: G7DA-28 (Z)D3 8A/240V (3-32V), OptoDevice:Finder_34.81, F.Cu at (133.5, 93.4)
- PS1: footprint Converter_ACDC:CONV_HLK-5M05 -> HLK-5M05:CONV_HLK-5M05
- R1: value 0R_0603 -> 10K; footprint PCM_Resistor_SMD_AKL:R_1206_3216Metric -> Resistor_SMD:R_1206_3216Metric; moved to B.Cu
- R2: value 0R_0603 -> ?; footprint PCM_Resistor_SMD_AKL:R_1206_3216Metric -> Resistor_SMD:R_1206_3216Metric; moved to B.Cu
- U1: value ESP32_DevKit_V1_DOIT -> ESP32-WROOM-E; footprint esp32_devkit_v1_doit:esp32_devkit_v1_doit -> Espressif:ESP32-WROOM-32E
- moved R1 53.2 mm to (117.7, 106.0), turned to 180 degrees
- moved REF** 50.0 mm to (158.7, 141.2)
- moved R2 47.6 mm to (117.7, 110.0), turned to 180 degrees
- moved C6 37.6 mm to (137.6, 118.2)
- moved J3 26.8 mm to (133.7, 111.2), turned to 180 degrees
- moved U1 21.7 mm to (151.8, 89.2), turned to -90 degrees
- moved J4 20.1 mm to (137.7, 111.2), turned to 180 degrees
- moved J6 17.1 mm to (153.9, 65.0), turned to 0 degrees
- moved J5 14.1 mm to (141.7, 111.2), turned to 180 degrees
- moved RVe1 11.3 mm to (128.7, 67.2), turned to -90 degrees
- moved PS1 8.14 mm to (118.2, 104.7), turned to 90 degrees
- moved FL1 4.44 mm to (121.2, 81.2)
- moved C5 1.77 mm to (117.7, 65.2)
- renumbered C1 to C5, C2 to C6
Connections:
- net HLK-AC1/J2-2 renamed Net-(PS1-AC2)
- net HLK-AC2/J1-2 renamed Net-(PS1-AC1)
- net J1-1/J2-1 renamed Net-(J1-Pin_1)
- net J1-2 renamed SSD-1
- C6 pad 1: +3V -> +3.3V
- J2 pad 2: Реле-выход/J2-1 -> SSD-2
- J3 pad 2: +3V -> +3.3V
- J4 pad 2: +3V -> +3.3V
- J5 pad 2: +3V -> +3.3V
- J6 pad 1: +3V -> +3.3V
- PS1 pad 4: +3V -> +3.3V
- R1 pad 1: Net-(U1-IO4) -> +3.3V
- R1 pad 2: Net-(D3-A) -> EN
- R2 pad 1: Net-(U1-IO5) -> Net-(C4-Pad1)
- R2 pad 2: Net-(D2-A) -> EN
- U1 pad 1: unconnected-(U1-EN-Pad1) -> GND
- U1 pad 13: unconnected-(U1-IO13-Pad13) -> TMS
- U1 pad 14: GND -> TDI
- U1 pad 15: unconnected-(U1-VIN-Pad15) -> GND
- U1 pad 16: +3V -> TCK
- U1 pad 17: GND -> (no net)
- U1 pad 18: Net-(U1-IO15) -> (no net)
- U1 pad 19: unconnected-(U1-IO2-Pad19) -> (no net)
- U1 pad 2: unconnected-(U1-SENSOR_VP-Pad2) -> +3.3V
- U1 pad 20: Net-(U1-IO4) -> (no net)
- U1 pad 21: unconnected-(U1-IO16-Pad21) -> (no net)
- U1 pad 22: unconnected-(U1-IO17-Pad22) -> (no net)
- U1 pad 23: Net-(U1-IO5) -> TDO
- U1 pad 25: unconnected-(U1-IO19-Pad25) -> GPIO0
- U1 pad 26: SDA -> unconnected-(U1-ADC2_CH0/GPIO4-Pad26)
- U1 pad 29: SCL -> unconnected-(U1-GPIO5-Pad29)
- U1 pad 3: unconnected-(U1-SENSOR_VN-Pad3) -> EN
- U1 pad 6: RELEAY -> GPIO34
Routing:
- net SDA: track 125.0 -> 0.00 mm
- net SCL: track 118.3 -> 0.00 mm
- net GND: track 48.9 -> 0.00 mm
- net SSD-1: track 45.9 -> 0.00 mm
- net ~220: track 45.5 -> 0.00 mm
- net Net-(PS1-AC1): track 40.5 -> 0.00 mm
- net Net-(D5-K): track 36.7 -> 0.00 mm
- net Net-(PS1-AC2): track 28.1 -> 0.00 mm
- net Реле-выход/J2-1: track 25.8 -> 0.00 mm
- net Net-(D2-A): track 21.7 -> 0.00 mm
- net Net-(D1-A): track 21.6 -> 0.00 mm
- net Net-(U1-IO5): track 19.6 -> 0.00 mm
- net Net-(D3-A): track 15.6 -> 0.00 mm
- net RELEAY: track 11.9 -> 0.00 mm
- net Net-(U1-IO4): track 10.6 -> 0.00 mm
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- added copper zone on B.Cu, net +3.3V
- removed copper zone on B.Cu, net +3V
Other:
- board text added: "RX"
- board text added: "TCK"
- board text added: "TDI"
- board text added: "TDO"
- board text added: "TMS"
- board text added: "TX"
- board text removed: "ERR"
- board text removed: "IOTV ID-5"
- board text removed: "TCP"
- board text removed: "WIFI"
- board text removed: "rev. 1.1"

Commit message: pcb id5 rev1.2
Other:
- board text added: "Boot"
- board text added: "En"
Changed lines of the file:
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@@
+    (effects (font (size 1 1) (thickness 0.15)) (justify left bottom))
+  )
+  (gr_text "Boot" (at 155.3464 115.3668) (layer "F.SilkS")
     (effects (font (size 1 1) (thickness 0.15)) (justify left bottom))
   )
@@
   )
   (gr_text "SCL" (at 144.194 104.204) (layer "F.SilkS")
+    (effects (font (size 1 1) (thickness 0.15)) (justify left bottom))
+  )
+  (gr_text "En" (at 146.3548 115.4176) (layer "F.SilkS")
     (effects (font (size 1 1) (thickness 0.15)) (justify left bottom))
   )
@@
   (segment (start 157.444 55.399) (end 157.444 52.669) (width 2.5) (layer "B.Cu") (net 9))
   (zone (net 1) (net_name "GND") (layer "F.Cu") (hatch edge 0.5)
-    (connect_pads (clearance 0.25))
+    (connect_pads (clearance 0.6))
     (min_thickness 0.25) (filled_areas_thickness no)
     (fill yes (thermal_gap 0.5) (thermal_bridge_width 0.5) (smoothing chamfer))
@@
         (xy 105.671518 122.104)
         (xy 104.144 121.425518)
-      )
-    )
-  )
-  (zone (net 0) (net_name "") (layers "F&B.Cu") (hatch edge 0.5)
-    (connect_pads (clearance 0))
-    (min_thickness 0.25) (filled_areas_thickness no)
-    (keepout (tracks allowed) (vias allowed) (pads allowed) (copperpour not_allowed) (footprints allowed))
-    (fill (thermal_gap 0.5) (thermal_bridge_width 0.5))
-    (polygon
-      (pts
-        (xy 104.14 50.804)
-        (xy 104.136211 -7.414)
-        (xy 117.598 -7.414)
-        (xy 117.598 -3.28937)
-        (xy 117.590205 0.75)
-        (xy 131.54 14.25)
-        (xy 134.54 14.25)
-        (xy 144.29 14.25)
-        (xy 169.54 14.25)
-        (xy 169.54 41.642)
-        (xy 169.54 50.804)
       )
     )
@@
   (zone (net 2) (net_name "+3.3V") (layer "B.Cu") (hatch edge 0.5)
     (priority 1)
-    (connect_pads (clearance 0.25))
+    (connect_pads (clearance 0.6))
     (min_thickness 0.25) (filled_areas_thickness no)
     (fill yes (thermal_gap 0.5) (thermal_bridge_width 0.5))

Commit message: pcb id5 rev 1.2
Parts:
- removed J7: JTAG, Connector_PinHeader_2.54mm:PinHeader_1x04_P2.54mm_Vertical
- C1, C2, C3, C4, R1, R2: moved to F.Cu
- moved logo 57.0 mm to (118.7, 100.6)
- moved C2 50.6 mm to (161.0, 73.7), turned to 180 degrees
- moved R1 50.2 mm to (160.0, 79.0), turned to 90 degrees
- moved C1 48.3 mm to (165.4, 79.0)
- moved C4 40.2 mm to (149.9, 117.3), turned to 180 degrees
- moved R2 37.5 mm to (153.0, 122.8), turned to 90 degrees
- moved C3 36.6 mm to (156.0, 122.8)
- moved J8 14.3 mm to (163.2, 114.0)
- moved SW2 5.56 mm to (162.0, 122.0)
- moved C6 4.22 mm to (137.6, 122.4)
- moved SW1 3.04 mm to (146.0, 122.0)
- moved C5 2.79 mm to (117.7, 68.0)
- moved J3 2.79 mm to (133.7, 114.0)
- moved J4 2.79 mm to (137.7, 114.0)
- moved J5 2.79 mm to (141.7, 114.0)
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- renumbered REF** to logo
Connections:
- FL1 pad 1: Net-(PS1-AC2) -> Net-(PS1-AC1)
- FL1 pad 4: Net-(PS1-AC1) -> Net-(PS1-AC2)
- J8 pad 1: +3.3V -> GND
- J8 pad 2: U0TX -> U0RX
- J8 pad 3: U0RX -> U0TX
- J8 pad 4: GND -> +3.3V
- U1 pad 13: TMS -> unconnected-(U1-MTMS/GPIO14/ADC2_CH6-Pad13)
- U1 pad 14: TDI -> unconnected-(U1-MTDI/GPIO12/ADC2_CH5-Pad14)
- U1 pad 16: TCK -> unconnected-(U1-MTCK/GPIO13/ADC2_CH4-Pad16)
- U1 pad 23: TDO -> unconnected-(U1-MTDO/GPIO15/ADC2_CH3-Pad23)
Routing:
- net SDA: track 0.00 -> 66.1 mm, vias 0 -> 1
- net SCL: track 0.00 -> 54.9 mm, vias 0 -> 1
- net EN: track 0.00 -> 49.3 mm, vias 0 -> 2
- net SSD-1: track 0.00 -> 44.8 mm
- net ~220: track 0.00 -> 38.4 mm
- net GPIO0: track 0.00 -> 32.5 mm
- net GPIO34: track 0.00 -> 28.8 mm
- net +3.3V: track 0.00 -> 28.6 mm
- net SSD-2: track 0.00 -> 27.4 mm
- net Net-(C4-Pad1): track 0.00 -> 15.9 mm
- net U0RX: track 0.00 -> 14.6 mm
- net U0TX: track 0.00 -> 12.3 mm
- net Net-(PS1-AC2): track 0.00 -> 9.76 mm
- net Net-(PS1-AC1): track 0.00 -> 6.72 mm
- removed copper zone on B.Cu, net ~220
Other:
- board size 83.1 x 77.8 mm -> 69.4 x 77.8 mm
- board text added: "IOTV ID-5"
- board text added: "rev. 1.2"
- board text removed: "TCK"
- board text removed: "TDI"
- board text removed: "TDO"
- board text removed: "TMS"
