File: IOTV/pcb/IOTV_id4/id4/untitled.kicad_sch (KiCad schematic)
At the start: 30 parts, among them Q1 S8050, Q10 S8050, Q11 S8050, Q12 S8050, Q2 S8050, Q3 S8050, Q7 S8050, Q8 S8050, Q9 S8050

Commit message: id4
pcd docs MK
Parts:
- added D1, D4: LED_RGBA, symbol Device:LED_RGBA
- added Q1, Q10, Q11, Q12, Q2, Q3: S8050, Package_TO_SOT_THT:TO-92_Inline, symbol Transistor_BJT:S8050
- added R1, R19, R2, R20: 5, symbol Device:R
- added R21, R3: 65, symbol Device:R
- added R22, R23, R24, R4, R5, R6: 100, symbol Device:R
Connections:
- net GND: now also Q1.1 (E), Q10.1 (E), Q11.1 (E), Q12.1 (E), Q2.1 (E), Q3.1 (E)
- net GPIO_12: now also R22.1; no longer R16.1
- net GPIO_13: now also R6.1; no longer R17.1
- net GPIO_14: now also R23.1; no longer R24.1
- net GPIO_23: now also R5.1; no longer R18.1
- net GPIO_27: now also R24.1; no longer R23.1
- net VCC_3.3: now also D1.4 (A), D4.4 (A)
- net at R15.1: now also D3.3 (BK); no longer D3.1 (RK)
- net at R19.1: now also D4.1 (RK); no longer D4.3 (BK)
- net at R1.1: now also D1.1 (RK); no longer D1.3 (BK)
- net at R3.1: now also D1.3 (BK); no longer D1.1 (RK)
- net at R21.1: now also D4.3 (BK); no longer D4.1 (RK)
- net at R13.1: now also D3.1 (RK); no longer D3.3 (BK)
- net GPIO_25 renamed GPIO_4
- net GPIO_26 renamed GPIO_16
- net GPIO_32 renamed GPIO_15
- net GPIO_33 renamed GPIO_2
- new net: D4.3 (BK), R21.1
- new net: Q12.3 (C), R21.2
- new net: D1.1 (RK), R1.1
- new net: D1.2 (GK), R2.1
- new net: D1.3 (BK), R3.1
- new net: Q3.3 (C), R2.2
- new net: Q12.2 (B), R24.2
- new net: Q1.3 (C), R1.2
- new net: D4.1 (RK), R19.1
- new net: D4.2 (GK), R20.1
- new net: Q1.2 (B), R4.2
- new net: Q3.2 (B), R5.2
- new net: Q10.2 (B), R22.2
- new net: Q11.3 (C), R20.2
- new net: Q10.3 (C), R19.2
- new net: Q2.3 (C), R3.2
- new net: Q11.2 (B), R23.2
- new net: Q2.2 (B), R6.2
- new net GPIO_17: R23.1
- new net GPIO_18: R16.1
- new net GPIO_19: R17.1
- new net GPIO_21: R18.1
- new net GPIO_22: R4.1
- new net GPIO_5: R24.1
Other:
- note added: "LED 0"
- note added: "LED 4"
- moved on the sheet: D1, D3, D4

Commit message: pcb id4
Parts:
- D1, D3, D4: footprint (none) -> LED_THT:LED_D5.0mm-4_RGB
- Q1, Q10, Q11, Q12, Q2, Q3, Q7, Q8, Q9: footprint Package_TO_SOT_THT:TO-92_Inline -> Package_TO_SOT_SMD:SOT-23
- R1, R13, R19: value 5 -> 150; footprint (none) -> Resistor_SMD:R_1206_3216Metric
- R14, R2, R20: value 5 -> 330; footprint (none) -> Resistor_SMD:R_1206_3216Metric
- R15, R21, R3: value 65 -> 100; footprint (none) -> Resistor_SMD:R_1206_3216Metric
- R16, R17, R18, R22, R23, R24, R4, R5, R6: footprint (none) -> Resistor_SMD:R_1206_3216Metric
Connections:
- net GPIO_16 renamed GPIO_33
- net GPIO_17 renamed GPIO_32
- net VCC_3.3 renamed VCC_5
Other:
- company: (none) -> Вербкин М.С.
- title: (none) -> IOTV_id4 LEDS
