File: IOTV/pcb/IOTV_id5/1.2/IOTV.kicad_pcb (KiCad board)
At the start: 2 copper layers, 69.4 x 77.8 mm, 24 parts, among them J1 Screw_Terminal_01x02, J2 Screw_Terminal_01x02, J3 Conn_01x04, J4 Conn_01x04, J5 Conn_01x04, J6 Conn_01x05, J8 UART, SW1 RST, SW2 Boot, U1 ESP32-WROOM-E, U2 G7DA-28 (Z)D3 8A/240V (3-32V)

Commit message: pcb id5 rev 1.2
Parts:
- C1, C2, R1: moved to B.Cu
- U2: footprint OptoDevice:Finder_34.81 -> Library:G7DA-28
- moved J8 36.7 mm to (150.7, 79.5)
- moved C2 23.1 mm to (158.0, 96.5), turned to -90 degrees
- moved R1 18.6 mm to (153.8, 96.5), turned to -90 degrees
- moved C1 18.1 mm to (161.5, 96.7)
- moved U2 17.7 mm to (138.8, 79.2), turned to -90 degrees
- moved U1 11.5 mm to (156.9, 102.3), turned to 0 degrees
- moved J3 11.3 mm to (134.0, 102.7), turned to 90 degrees
- moved J5 8.36 mm to (134.0, 110.7), turned to 90 degrees
- moved J4 8.19 mm to (134.0, 106.7), turned to 90 degrees
- moved J6 1.82 mm to (155.5, 68.8), turned to 90 degrees
- moved PS1 0.53 mm to (118.3, 107.0)
- moved C6 0.36 mm to (137.6, 122.1)
Connections:
- J8 pad 2: U0RX -> U0TX
- J8 pad 3: U0TX -> U0RX
Routing:
- net GND: track 0.00 -> 26.7 mm, vias 0 -> 2
- net +3.3V: track 28.6 -> 6.21 mm, vias 0 -> 1
- net U0RX: track 14.6 -> 36.3 mm
- net U0TX: track 12.3 -> 32.7 mm
- net GPIO0: track 32.5 -> 14.9 mm
- net SDA: track 66.1 -> 82.9 mm
- net SCL: track 54.9 -> 70.0 mm
- net EN: track 49.3 -> 35.3 mm, vias 2 -> 1
- net GPIO34: track 28.8 -> 20.9 mm
- net SSD-1: track 44.8 -> 52.6 mm

Commit message: pcb
Parts:
- moved J3 12.2 mm to (133.1, 114.9), turned to 180 degrees
- moved J4 8.76 mm to (137.1, 114.9), turned to 180 degrees
- moved J5 8.24 mm to (141.1, 114.9), turned to 180 degrees
- moved U2 1.56 mm to (139.3, 77.7)
Routing:
- net GPIO34: track 20.9 -> 14.2 mm
- net SDA: track 82.9 -> 88.4 mm
- net SCL: track 70.0 -> 72.4 mm
- net SSD-2: track 27.0 -> 28.4 mm
- net SSD-1: track 52.6 -> 54.1 mm

Commit message: pcb id5 rev 1.2 ssr
Parts:
- removed logo: KiCad-Logo2_5mm_SilkScreen, Symbol:KiCad-Logo2_5mm_SilkScreen
