File: IOTV/pcb/IOTV_id5/1.2/IOTV.kicad_pcb (KiCad board)
At the start: 2 copper layers, 69.4 x 77.8 mm, 23 parts, among them J1 Screw_Terminal_01x02, J2 Screw_Terminal_01x02, J3 Conn_01x04, J4 Conn_01x04, J5 Conn_01x04, J6 Conn_01x05, J8 UART, SW1 RST, SW2 Boot, U1 ESP32-WROOM-E, U2 G7DA-28 (Z)D3 8A/240V (3-32V)

Commit message: MK id5 1.1
Parts:
- added Q1: S8050, Package_TO_SOT_SMD:SOT-23, B.Cu at (139.6, 87.5)
Connections:
- U1 pad 6: GPIO34 -> unconnected-(U1-GPIO34/ADC1_CH6-Pad6)
- U1 pad 8: unconnected-(U1-32K_XP/GPIO32/ADC1_CH4-Pad8) -> GPIO32
- U2 pad A1: GPIO34 -> ssr+
Routing:
- net GPIO32: track 0.00 -> 19.7 mm, vias 0 -> 1
- net GPIO34: track 14.2 -> 0.00 mm
- net ssr+: track 0.00 -> 3.95 mm
- net SDA: track 88.4 -> 90.7 mm
