File: IOTV/pcb/IOTV_id5/1.2/IOTV.kicad_pcb (KiCad board)
At the start: 2 copper layers, 69.4 x 77.8 mm, 24 parts, among them J1 Screw_Terminal_01x02, J2 Screw_Terminal_01x02, J3 Conn_01x04, J4 Conn_01x04, J5 Conn_01x04, J6 Conn_01x05, J8 UART, Q1 S8050, SW1 RST, SW2 Boot, U1 ESP32-WROOM-E, U2 G7DA-28 (Z)D3 8A/240V (3-32V)

Commit message: удаление старых файлов
Routing:
- net +3.3V: track 6.21 -> 2.94 mm
Changed lines of the file:
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@@
   (segment (start 148.195 96.52) (end 151.13 96.52) (width 0.5) (layer "F.Cu") (net 2))
   (via (at 151.13 96.52) (size 0.8) (drill 0.4) (layers "F.Cu" "B.Cu") (free) (net 2))
-  (segment (start 153.797 95.0575) (end 152.5925 95.0575) (width 0.5) (layer "B.Cu") (net 2))
-  (segment (start 152.5925 95.0575) (end 151.13 96.52) (width 0.5) (layer "B.Cu") (net 2))
   (segment (start 121.171 74.07675) (end 121.171 71.475) (width 2.5) (layer "B.Cu") (net 3))
   (segment (start 124.61525 74.07675) (end 128.694 69.998) (width 2.5) (layer "B.Cu") (net 3))
